Commit message: cmd_publisher.py updated

File: description_dual/urdf/base.urdf.xacro (robot description, xacro)
@@ -8,5 +8,24 @@
     <xacro:include filename="$(find description_dual)/urdf/materials.urdf.xacro"/>
     <!-- Base footprint -->
-    <link name="base_footprint"/>
+    <link name="base_footprint">
+        <inertial>
+            <origin xyz="0 0 0" rpy="0 0 0" />
+            <mass value="0.1" />
+            <inertia ixx="1.0" ixy="0.0" ixz="0.0" iyy="1.0" iyz="0.0" izz="0.0" />
+        </inertial>
+        <visual>
+            <origin xyz="0 0 0" rpy="0 0 0" />
+            <geometry>
+                <box size="0.001 0.001 0.001"/>
+            </geometry>
+            <material name="material_red"/>
+        </visual>
+        <collision>
+        <origin xyz="0 0 0" rpy="0 0 0" />
+            <geometry>
+                <box size="0.001 0.001 0.001"/>
+            </geometry>
+        </collision>
+    </link>
     <joint name="base_joint" type="fixed">
         <parent link="base_footprint"/>

Commit message: pkg arrangemnet

File: description_dual/urdf/base.urdf.xacro (robot description, xacro)
@@ -7,22 +7,31 @@
     <xacro:include filename="$(find description_dual)/urdf/base.gazebo.xacro"/>
     <xacro:include filename="$(find description_dual)/urdf/materials.urdf.xacro"/>
-    <!-- Base footprint -->
-    <link name="base_footprint">
-        <inertial>
-            <origin xyz="0 0 0" rpy="0 0 0" />
-            <mass value="0.1" />
-            <inertia ixx="1.0" ixy="0.0" ixz="0.0" iyy="1.0" iyz="0.0" izz="0.0" />
-        </inertial>
-        <visual>
-            <origin xyz="0 0 0" rpy="0 0 0" />
-            <geometry>
-                <box size="0.001 0.001 0.001"/>
-            </geometry>
-            <material name="material_red"/>
+    <!-- Odom -->
+    <link name="odom"/>
+     <!-- Base footprint -->
+    <link name="base_footprint"/>
+    <joint name="odom_joint" type="fixed">
+        <parent link="odom"/>
+        <child link="base_footprint"/>
+        <origin xyz="0.0 0.0 0.0" rpy="0 0 0"/>
+    </joint>
+    <!-- Base link -->
+    <link name="base_link">
+        <inertial>
+            <origin xyz="0 0 0" rpy="0 0 0" />
+            <mass value="13.2312244818196" />
+            <inertia ixx="0.967053548924663" ixy="0" ixz="0" iyy="1.30612724440363" iyz="0" izz="0.962964405480844" />
+        </inertial>
+        <visual>
+            <origin xyz="0 0 0" rpy="0 0 0" />
+            <geometry>
+                <mesh filename="package://description_dual/meshes/base_link.STL" />
+            </geometry>
+            <material name="material_light_grey"/>
         </visual>
         <collision>
         <origin xyz="0 0 0" rpy="0 0 0" />
             <geometry>
-                <box size="0.001 0.001 0.001"/>
+                <mesh filename="package://description_dual/meshes/base_link.STL" />
             </geometry>
         </collision>
@@ -33,25 +42,4 @@
         <origin xyz="0.0 0.0 0.0" rpy="0 0 0"/>
     </joint>
-    <!-- Base link -->
-    <link name="base_link">
-        <inertial>
-            <origin xyz="0 0 0" rpy="0 0 0" />
-            <mass value="13.2312244818196" />
-            <inertia ixx="0.967053548924663" ixy="0" ixz="0" iyy="1.30612724440363" iyz="0" izz="0.962964405480844" />
-        </inertial>
-        <visual>
-            <origin xyz="0 0 0" rpy="0 0 0" />
-            <geometry>
-                <mesh filename="package://description_dual/meshes/base_link.STL" />
-            </geometry>
-            <material name="material_light_grey"/>
-        </visual>
-        <collision>
-        <origin xyz="0 0 0" rpy="0 0 0" />
-            <geometry>
-                <mesh filename="package://description_dual/meshes/base_link.STL" />
-            </geometry>
-        </collision>
-    </link>
     <!-- Back right wheel -->
     <link name="br_wheel_link">
