Commit message: version 0.1

File: description_dual/urdf/base.gazebo.xacro (robot description, xacro)
@@ -32,5 +32,5 @@
         <material>Gazebo/FlatBlack</material>
     </gazebo>
-    <gazebo>
+    <!-- <gazebo>
       <plugin name="p3d_base_controller" filename="libgazebo_ros_p3d.so">
         <alwaysOn>true</alwaysOn>
@@ -43,5 +43,5 @@
         <rpyOffsets>0 0 0</rpyOffsets>
       </plugin>
-    </gazebo>
+    </gazebo> -->
     <gazebo>
         <plugin name="imu_plugin" filename="libgazebo_ros_imu.so">

File: description_dual/urdf/base.urdf.xacro (robot description, xacro)
@@ -28,4 +28,25 @@
         </collision>
     </link>
+    <!-- Base link -->
+    <link name="base_link">
+        <inertial>
+            <origin xyz="0 0 0" rpy="0 0 0" />
+            <mass value="13.2312244818196" />
+            <inertia ixx="0.967053548924663" ixy="0" ixz="0" iyy="1.30612724440363" iyz="0" izz="0.962964405480844" />
+        </inertial>
+        <visual>
+            <origin xyz="0 0 0" rpy="0 0 0" />
+            <geometry>
+                <mesh filename="package://description_dual/meshes/base_link.STL" />
+            </geometry>
+            <material name="material_light_grey"/>
+        </visual>
+        <collision>
+        <origin xyz="0 0 0" rpy="0 0 0" />
+            <geometry>
+                <mesh filename="package://description_dual/meshes/base_link.STL" />
+            </geometry>
+        </collision>
+    </link>
     <joint name="base_joint" type="fixed">
         <parent link="base_footprint"/>
@@ -33,25 +54,4 @@
         <origin xyz="0.0 0.0 0.0" rpy="0 0 0"/>
     </joint>
-    <!-- Base link -->
-    <link name="base_link">
-        <inertial>
-            <origin xyz="0 0 0" rpy="0 0 0" />
-            <mass value="13.2312244818196" />
-            <inertia ixx="0.967053548924663" ixy="0" ixz="0" iyy="1.30612724440363" iyz="0" izz="0.962964405480844" />
-        </inertial>
-        <visual>
-            <origin xyz="0 0 0" rpy="0 0 0" />
-            <geometry>
-                <mesh filename="package://description_dual/meshes/base_link.STL" />
-            </geometry>
-            <material name="material_light_grey"/>
-        </visual>
-        <collision>
-        <origin xyz="0 0 0" rpy="0 0 0" />
-            <geometry>
-                <mesh filename="package://description_dual/meshes/base_link.STL" />
-            </geometry>
-        </collision>
-    </link>
     <!-- Back right wheel -->
     <link name="br_wheel_link">

Commit message: pkg changinged

File: description_dual/urdf/base.gazebo.xacro (robot description, xacro)
@@ -77,5 +77,5 @@
         <sensor type="gpu_ray" name="lds_lfcd_sensor">
         <pose>0 0 0 0 0 0</pose>
-        <visualize>false</visualize>
+        <visualize>true</visualize>
         <update_rate>50</update_rate>
         <ray>
@@ -102,4 +102,6 @@
             <topicName>scan</topicName>
             <frameName>base_scan</frameName>
+            <gaussianNoise>0.01</gaussianNoise>
+            <updateRate>20.0</updateRate>
         </plugin>
         </sensor>
@@ -110,5 +112,5 @@
         <sensor type="ray" name="sonar_front_sensor">
         <pose>0 0 0 0 0 0</pose>
-        <visualize>false</visualize>
+        <visualize>true</visualize>
         <update_rate>50</update_rate>
         <ray>
@@ -138,4 +140,6 @@
             <fov>0.5</fov>
             <radiation>ultrasound</radiation>
+            <gaussianNoise>0.01</gaussianNoise>
+            <updateRate>20.0</updateRate>
         </plugin>
       </sensor>
@@ -145,5 +149,5 @@
         <sensor type="ray" name="sonar_rear_sensor">
         <pose>0 0 0 0 0 0</pose>
-        <visualize>false</visualize>
+        <visualize>true</visualize>
         <update_rate>50</update_rate>
         <ray>
@@ -173,4 +177,6 @@
             <fov>0.5</fov>
             <radiation>ultrasound</radiation>
+            <gaussianNoise>0.01</gaussianNoise>
+            <updateRate>20.0</updateRate>
         </plugin>
       </sensor>
@@ -180,5 +186,5 @@
         <sensor type="ray" name="sonar_left_sensor">
         <pose>0 0 0 0 0 0</pose>
-        <visualize>false</visualize>
+        <visualize>true</visualize>
         <update_rate>50</update_rate>
         <ray>
@@ -208,4 +214,6 @@
             <fov>0.5</fov>
             <radiation>ultrasound</radiation>
+            <gaussianNoise>0.01</gaussianNoise>
+            <updateRate>20.0</updateRate>
         </plugin>
       </sensor>
@@ -215,5 +223,5 @@
         <sensor type="ray" name="sonar_right_sensor">
         <pose>0 0 0 0 0 0</pose>
-        <visualize>false</visualize>
+        <visualize>true</visualize>
         <update_rate>50</update_rate>
         <ray>
@@ -243,4 +251,6 @@
             <fov>0.5</fov>
             <radiation>ultrasound</radiation>
+            <gaussianNoise>0.01</gaussianNoise>
+            <updateRate>20.0</updateRate>
         </plugin>
       </sensor>

File: description_dual/urdf/base.urdf.xacro (robot description, xacro)
@@ -7,13 +7,6 @@
     <xacro:include filename="$(find description_dual)/urdf/base.gazebo.xacro"/>
     <xacro:include filename="$(find description_dual)/urdf/materials.urdf.xacro"/>
-    <!-- Odom -->
-    <link name="odom"/>
-     <!-- Base footprint -->
+    <!-- Base footprint -->
     <link name="base_footprint"/>
-    <joint name="odom_joint" type="fixed">
-        <parent link="odom"/>
-        <child link="base_footprint"/>
-        <origin xyz="0.0 0.0 0.0" rpy="0 0 0"/>
-    </joint>
     <!-- Base link -->
     <link name="base_link">
